Commit message: done nav2 with cartographer

File: my_diff_drive_robot/urdf/lidar.xacro (robot description, xacro)
@@ -1,47 +1,60 @@
 <?xml version="1.0"?>
+<!-- lidar xacro -->
 <robot xmlns:xacro="http://ros.org/wiki/xacro">
-<xacro:macro name="laser" params="parent_link">
-  <link name="lidar_link">
-    <visual>
-      <geometry>
-        <cylinder radius="0.03" length="0.06"/>
-      </geometry>
-      <material name="blue"/>
-    </visual>
-    <collision>
-      <geometry>
-        <cylinder radius="0.03" length="0.06"/>
-      </geometry>
-    </collision>
-  </link>
-  <joint name="lidar_joint" type="fixed">
-    <parent link="${parent_link}"/>
-    <child link="lidar_link"/>
-    <origin xyz="0 0 0.2"/>
-  </joint>
-  <gazebo reference="lidar_link">
-    <sensor name="lidar" type="ray">
-      <pose> 0 0 0 0 0 0 </pose>
-      <visualize>true</visualize>
-      <update_rate>30</update_rate>
-      <ray>
-        <scan>
-          <horizontal>
-            <samples>720</samples>
-            <min_angle>-3.14</min_angle>
-            <max_angle>3.14</max_angle>
-          </horizontal>
-        </scan>
-        <range>
-          <min>0.1</min>
-          <max>8.0</max>
-        </range>
-      </ray>
-      <plugin name="lidar_controller" filename="libgazebo_ros2_laser.so">
-        <topicName>/scan</topicName>
-        <frameName>lidar_link</frameName>
-      </plugin>
-    </sensor>
-  </gazebo>
-</xacro:macro>
+  <xacro:macro name="laser" params="parent_link">
+    <link name="lidar_link">
+      <visual>
+        <geometry>
+          <cylinder radius="0.03" length="0.06" />
+        </geometry>
+        <material name="blue" />
+      </visual>
+      <collision>
+        <geometry>
+          <cylinder radius="0.03" length="0.06" />
+        </geometry>
+      </collision>
+    </link>
+    <joint name="lidar_joint" type="fixed">
+      <parent link="${parent_link}" />
+      <child link="lidar_link" />
+      <origin xyz="0 0 0.2" />
+    </joint>
+    <!-- The Gazebo sensor definition attached to lidar_link -->
+    <gazebo reference="lidar_link">
+      <sensor name="lidar" type="ray">
+        <pose>0 0 0 0 0 0</pose>
+        <always_on>true</always_on>
+        <visualize>true</visualize>
+        <update_rate>5</update_rate>
+        <ray>
+          <scan>
+            <horizontal>
+              <samples>720</samples>
+              <!-- <resolution>1.00000</resolution> -->
+              <min_angle>-3.14</min_angle>
+              <max_angle>3.14</max_angle>
+            </horizontal>
+          </scan>
+          <range>
+            <min>0.1</min>
+            <max>10.0</max>
+            <resolution>0.015000</resolution>
+          </range>
+          <noise>
+            <type>gaussian</type>
+            <mean>0.0</mean>
+            <stddev>0.01</stddev>
+          </noise>
+        </ray>
+        <plugin name="scan" filename="libgazebo_ros_ray_sensor.so">
+          <ros>
+            <remapping>~/out:=scan</remapping>
+          </ros>
+          <output_type>sensor_msgs/LaserScan</output_type>
+          <frame_name>lidar_link</frame_name>
+        </plugin>
+      </sensor>
+    </gazebo>
+  </xacro:macro>
 </robot>

File: my_diff_drive_robot/urdf/my_diff_drive.urdf.xacro (robot description, xacro)
@@ -1,156 +1,154 @@
 <?xml version="1.0"?>
+<!-- my_diff_drive.urdf.xacro -->
 <robot name="my_diff_drive_robot" xmlns:xacro="http://ros.org/wiki/xacro">
-    <!-- Include macros -->
-    <xacro:include filename="$(find my_diff_drive_robot)/urdf/inertial_macros.xacro" />
-    <xacro:include filename="$(find my_diff_drive_robot)/urdf/lidar.xacro" />
-    <xacro:arg name="robot_namespace" default="/" />
-    <!-- Materials -->
-    <material name="white">
-        <color rgba="1 1 1 1" />
-    </material>
-    <material name="orange">
-        <color rgba="1 0.3 0.1 1" />
-    </material>
-    <material name="blue">
-        <color rgba="0.2 0.2 1 1" />
-    </material>
-    <material name="black">
-        <color rgba="0 0 0 1" />
-    </material>
-    <!-- Base Link -->
-    <link name="base_link" />
-    <!-- Chassis -->
-    <joint name="chassis_joint" type="fixed">
-        <parent link="base_link" />
-        <child link="chassis" />
-        <origin xyz="0 0 0" />
-    </joint>
-    <link name="chassis">
-        <visual>
-            <origin xyz="0 0 0.075" />
-            <geometry>
-                <box size="0.3 0.3 0.15" />
-            </geometry>
-            <material name="white" />
-        </visual>
-        <collision>
-            <origin xyz="0 0 0.075" />
-            <geometry>
-                <box size="0.3 0.3 0.15" />
-            </geometry>
-        </collision>
-        <xacro:inertial_box mass="0.5" x="0.3" y="0.3" z="0.15">
-            <origin xyz="0 0 0.075" />
-        </xacro:inertial_box>
-    </link>
-    <!-- Left Wheel -->
-    <link name="left_wheel_link">
-        <visual>
-            <geometry>
-                <cylinder radius="0.05" length="0.04" />
-            </geometry>
-            <material name="black" />
-        </visual>
-        <collision>
-            <geometry>
-                <cylinder radius="0.05" length="0.04" />
-            </geometry>
-        </collision>
-        <xacro:inertial_cylinder mass="0.1" length="0.04" radius="0.05">
-            <origin xyz="0 0 0" />
-        </xacro:inertial_cylinder>
-    </link>
-    <joint name="left_wheel_joint" type="continuous">
-        <parent link="base_link" />
-        <child link="left_wheel_link" />
-        <origin xyz="0 0.175 0" rpy="-${pi/2} 0 0" />
-        <axis xyz="0 0 1" />
-        <dynamics damping="0.5" friction="10.0" />
-    </joint>
-    <!-- Right Wheel -->
-    <link name="right_wheel_link">
-        <visual>
-            <geometry>
-                <cylinder radius="0.05" length="0.04" />
-            </geometry>
-            <material name="black" />
-        </visual>
-        <collision>
-            <geometry>
-                <cylinder radius="0.05" length="0.04" />
-            </geometry>
-        </collision>
-        <xacro:inertial_cylinder mass="0.1" length="0.04" radius="0.05">
-            <origin xyz="0 0 0" />
-        </xacro:inertial_cylinder>
-    </link>
-    <joint name="right_wheel_joint" type="continuous">
-        <parent link="base_link" />
-        <child link="right_wheel_link" />
-        <origin xyz="0 -0.175 0" rpy="${pi/2} 0 0" />
-        <axis xyz="0 0 -1" />
-        <dynamics damping="0.5" friction="10.0" />
-    </joint>
-    <!-- Caster Wheel (front) -->
-    <joint name="caster_wheel_joint" type="fixed">
-        <parent link="chassis" />
-        <child link="caster_wheel_link" />
-        <origin xyz="0.14 0 0" />
-        <dynamics damping="0.0" friction="0.0" />
-    </joint>
-    <link name="caster_wheel_link">
-        <visual>
-            <geometry>
-                <sphere radius="0.05" />
-            </geometry>
-            <material name="black" />
-        </visual>
-        <collision>
-            <geometry>
-                <sphere radius="0.05" />
-            </geometry>
-        </collision>
-        <xacro:inertial_sphere mass="0.1" radius="0.05">
-            <origin xyz="0 0 0" />
-        </xacro:inertial_sphere>
-    </link>
-    <gazebo reference="caster_wheel_link">
-        <mu1 value="0.0" />
-        <mu2 value="0.0" />
-        <kp value="10000000.0" />
-        <kd value="1.0" />
-        <fdir1 value="1 0 0" />
-        <material>Gazebo/Grey</material>
-        <turnGravityOff>false</turnGravityOff>
-    </gazebo>
-    <!-- Insert the LiDAR sensor macro -->
-    <xacro:laser parent_link="chassis" />
-    <!-- Gazebo Plugin for Differential Drive -->
-    <gazebo>
-        <plugin name="diff_drive_controller" filename="libgazebo_ros_diff_drive.so">
-            <!-- Names of the joints -->
-            <left_joint>left_wheel_joint</left_joint>
-            <right_joint>right_wheel_joint</right_joint>
-            <!-- Topic on which velocity commands will be received -->
-            <command_topic>cmd_vel</command_topic>
-            <!-- Publish odometry on /odom -->
-            <odometry_topic>odom</odometry_topic>
-            <odometry_frame>odom</odometry_frame>
-            <publish_odom>true</publish_odom>
-            <publish_odom_tf>true</publish_odom_tf>
-            <publish_wheel_tf>true</publish_wheel_tf>
-            <!-- TF for odom->base_link transform -->
-            <robot_base_frame>base_link</robot_base_frame>
-            <!-- Wheel separation & radius (should match URDF) -->
-            <wheel_separation>0.35</wheel_separation>
-            <wheel_radius>0.05</wheel_radius>
-            <wheel_diameter>0.1</wheel_diameter>
-            <!-- Limits -->
-            <max_wheel_torque>200</max_wheel_torque>
-            <max_wheel_acceleration>10.0</max_wheel_acceleration>
-            <!-- Plugin parameters -->
-            <update_rate>50</update_rate>
-            <publish_tf>true</publish_tf>
-        </plugin>
-    </gazebo>
+  <!-- Include macros by relative path (assumes they are in the same folder) -->
+  <xacro:include filename="inertial_macros.xacro" />
+  <xacro:include filename="lidar.xacro" />
+  <!-- Materials -->
+  <material name="white">
+    <color rgba="1 1 1 1" />
+  </material>
+  <material name="black">
+    <color rgba="0 0 0 1" />
+  </material>
+  <material name="blue">
+    <color rgba="0.2 0.2 1 1" />
+  </material>
+  <!-- Base Link -->
+  <link name="base_link" />
+  <!-- Chassis -->
+  <joint name="chassis_joint" type="fixed">
+    <parent link="base_link" />
+    <child link="chassis" />
+    <origin xyz="0 0 0" />
+  </joint>
+  <link name="chassis">
+    <visual>
+      <origin xyz="0 0 0.075" />
+      <geometry>
+        <box size="0.3 0.3 0.15" />
+      </geometry>
+      <material name="white" />
+    </visual>
+    <collision>
+      <origin xyz="0 0 0.075" />
+      <geometry>
+        <box size="0.3 0.3 0.15" />
+      </geometry>
+    </collision>
+    <!-- Use your inertial macro -->
+    <xacro:inertial_box mass="0.5" x="0.3" y="0.3" z="0.15">
+      <origin xyz="0 0 0.075" />
+    </xacro:inertial_box>
+  </link>
+  <!-- Left Wheel -->
+  <link name="left_wheel_link">
+    <visual>
+      <geometry>
+        <cylinder radius="0.05" length="0.04" />
+      </geometry>
+      <material name="black" />
+    </visual>
+    <collision>
+      <geometry>
+        <cylinder radius="0.05" length="0.04" />
+      </geometry>
+    </collision>
+    <xacro:inertial_cylinder mass="0.1" length="0.04" radius="0.05">
+      <origin xyz="0 0 0" />
+    </xacro:inertial_cylinder>
+  </link>
+  <joint name="left_wheel_joint" type="continuous">
+    <parent link="base_link" />
+    <child link="left_wheel_link" />
+    <origin xyz="0 0.175 0" rpy="-${pi/2} 0 0" />
+    <axis xyz="0 0 1" />
+    <dynamics damping="0.5" friction="10.0" />
+  </joint>
+  <!-- Right Wheel -->
+  <link name="right_wheel_link">
+    <visual>
+      <geometry>
+        <cylinder radius="0.05" length="0.04" />
+      </geometry>
+      <material name="black" />
+    </visual>
+    <collision>
+      <geometry>
+        <cylinder radius="0.05" length="0.04" />
+      </geometry>
+    </collision>
+    <xacro:inertial_cylinder mass="0.1" length="0.04" radius="0.05">
+      <origin xyz="0 0 0" />
+    </xacro:inertial_cylinder>
+  </link>
+  <joint name="right_wheel_joint" type="continuous">
+    <parent link="base_link" />
+    <child link="right_wheel_link" />
+    <origin xyz="0 -0.175 0" rpy="${pi/2} 0 0" />
+    <axis xyz="0 0 -1" />
+    <dynamics damping="0.5" friction="10.0" />
+  </joint>
+  <!-- Caster Wheel -->
+  <joint name="caster_wheel_joint" type="fixed">
+    <parent link="chassis" />
+    <child link="caster_wheel_link" />
+    <origin xyz="0.14 0 0" />
+  </joint>
+  <link name="caster_wheel_link">
+    <visual>
+      <geometry>
+        <sphere radius="0.05" />
+      </geometry>
+      <material name="black" />
+    </visual>
+    <collision>
+      <geometry>
+        <sphere radius="0.05" />
+      </geometry>
+    </collision>
+    <xacro:inertial_sphere mass="0.1" radius="0.05">
+      <origin xyz="0 0 0" />
+    </xacro:inertial_sphere>
+  </link>
+  <gazebo reference="caster_wheel_link">
+    <mu1 value="0.0" />
+    <mu2 value="0.0" />
+  </gazebo>
+  <!-- Insert the LiDAR sensor macro (above the chassis) -->
+  <xacro:laser parent_link="base_link" />
+  <!-- Publish Joint States -->
+  <gazebo>
+    <plugin name="joint_state_publisher" filename="libgazebo_ros_joint_state_publisher.so">
+      <always_publish>true</always_publish>
+      <publish_default_positions>true</publish_default_positions>
+      <ros>
+        <remapping>~/out:=joint_states</remapping>
+      </ros>
+      <update_rate>30</update_rate>
+      <joint_name>left_wheel_joint</joint_name>
+      <joint_name>right_wheel_joint</joint_name>
+    </plugin>
+  </gazebo>
+  <!-- Diff Drive Plugin -->
+  <gazebo>
+    <plugin name="diff_drive_controller" filename="libgazebo_ros_diff_drive.so">
+      <left_joint>left_wheel_joint</left_joint>
+      <right_joint>right_wheel_joint</right_joint>
+      <command_topic>cmd_vel</command_topic>
+      <!-- <odometry_topic>odom</odometry_topic>
+      <odometry_frame>odom</odometry_frame>
+      <publish_odom>true</publish_odom>
+      <publish_odom_tf>true</publish_odom_tf> -->
+      <publish_wheel_tf>true</publish_wheel_tf>
+      <robot_base_frame>base_link</robot_base_frame>
+      <wheel_separation>0.35</wheel_separation>
+      <wheel_diameter>0.1</wheel_diameter>
+      <wheel_radius>0.05</wheel_radius>
+      <max_wheel_torque>200</max_wheel_torque>
+      <max_wheel_acceleration>10.0</max_wheel_acceleration>
+      <update_rate>50</update_rate>
+      <publish_tf>true</publish_tf>
+    </plugin>
+  </gazebo>
 </robot>

Commit message: update with mesh

File: my_diff_drive_robot/urdf/lidar.xacro (robot description, xacro)
@@ -6,5 +6,5 @@
       <visual>
         <geometry>
-          <cylinder radius="0.03" length="0.06" />
+          <cylinder radius="0.03" length="0.04" />
         </geometry>
         <material name="blue" />
@@ -12,5 +12,5 @@
       <collision>
         <geometry>
-          <cylinder radius="0.03" length="0.06" />
+          <cylinder radius="0.03" length="0.04" />
         </geometry>
       </collision>
@@ -19,5 +19,5 @@
       <parent link="${parent_link}" />
       <child link="lidar_link" />
-      <origin xyz="0 0 0.2" />
+      <origin xyz="0 0 0.14" />
     </joint>
     <!-- The Gazebo sensor definition attached to lidar_link -->
@@ -45,5 +45,5 @@
             <type>gaussian</type>
             <mean>0.0</mean>
-            <stddev>0.01</stddev>
+            <stddev>0.015</stddev>
           </noise>
         </ray>

File: my_diff_drive_robot/urdf/my_diff_drive.urdf_no_mesh.xacro (robot description, xacro)
@@ -5,5 +5,4 @@
   <xacro:include filename="inertial_macros.xacro" />
   <xacro:include filename="lidar.xacro" />
-  <!-- <xacro:property name="pi" value="3.141592653589793"/> -->
   <!-- Materials -->
   <material name="white">
@@ -15,7 +14,4 @@
   <material name="blue">
     <color rgba="0.2 0.2 1 1" />
-  </material>
-  <material name="light_black">
-    <color rgba="0.3 0.3 0.3 1" />
   </material>
   <!-- Base Link -->
@@ -29,23 +25,20 @@
   <link name="chassis">
     <visual>
-      <origin xyz="-0.1 0.1 0.0" rpy="0 0 ${pi/2}"/>
+      <origin xyz="0 0 0.05" />
       <geometry>
-        <mesh filename="package://my_diff_drive_robot/urdf/meshes/chassis.dae" scale="0.001 0.001 0.001"/>
+        <box size="0.25 0.25 0.10" />
       </geometry>
-      <material name="light_black" />
+      <material name="white" />
     </visual>
     <collision>
-       <origin xyz="-0.1 0.1 0.0" rpy="0 0 ${pi/2}"/>
+      <origin xyz="0 0 0.05" />
       <geometry>
-        <mesh filename="package://my_diff_drive_robot/urdf/meshes/chassis.dae" scale="0.001 0.001 0.001"/>
+        <box size="0.25 0.25 0.10" />
       </geometry>
     </collision>
-    <inertial>
-      <origin xyz="0 0 0" rpy="0 0 0" />
-      <mass value="1.3729096e+00" />
-      <inertia ixx="8.7002718e-03" ixy="-4.7576583e-05" ixz="1.1160499e-04"
-        iyy="8.6195418e-03" iyz="-3.5422299e-06"
-        izz="1.4612727e-02" />
-    </inertial>
+    <!-- Use your inertial macro -->
+    <xacro:inertial_box mass="0.5" x="0.25" y="0.25" z="0.10">
+      <origin xyz="0 0 0.05" />
+    </xacro:inertial_box>
   </link>
   <!-- Left Wheel -->
